File: custom_microbrics.kicad_pcb (KiCad board)
At the start: 2 copper layers, 20.2 x 20.2 mm, 2 parts, among them J1 Conn_01x03

Commit message: led module
Parts:
- removed J1: Conn_01x03, Connector_PinHeader_2.54mm:PinHeader_1x03_P2.54mm_Vertical
- added D1: LED, LED_THT:LED_D3.0mm, F.Cu at (148.6, 111.8)
- added R1: R_Small_US, Resistor_THT:R_Axial_DIN0207_L6.3mm_D2.5mm_P10.16mm_Horizontal, F.Cu at (156.2, 111.8)
Routing:
- net Net-(MB1-Pad3): track 12.8 -> 2.15 mm
- net Net-(D1-Pad2): track 0.00 -> 5.08 mm
- net Net-(D1-Pad1): track 13.0 -> 17.7 mm
- net Net-(MB1-Pad2): track 12.0 -> 10.3 mm
